Commit message: Update the urdf of panda robot arm

File: config/urdfs/panda.urdf (robot description, URDF)
Before this commit: robot panda, 12 links, 11 joints
Links:
- added link world
- link panda_hand: mass None -> 0.73; geometry collision mesh filename=package://franka_gazebo/meshes/collision/hand.stl; visual mesh filename=package://franka_gazebo/meshes/visual/hand.dae
- link panda_leftfinger: mass None -> 0.1; geometry collision mesh filename=package://franka_gazebo/meshes/collision/finger.stl; visual mesh filename=package://franka_gazebo/meshes/visual/finger.dae
- link panda_link0: mass None -> 2.92; geometry collision mesh filename=package://franka_gazebo/meshes/collision/link0.stl; visual mesh filename=package://franka_gazebo/meshes/visual/link0.dae
- link panda_link1: mass None -> 2.74; geometry collision mesh filename=package://franka_gazebo/meshes/collision/link1.stl; visual mesh filename=package://franka_gazebo/meshes/visual/link1.dae
- link panda_link2: mass None -> 2.74; geometry collision mesh filename=package://franka_gazebo/meshes/collision/link2.stl; visual mesh filename=package://franka_gazebo/meshes/visual/link2.dae
- link panda_link3: mass None -> 2.38; geometry collision mesh filename=package://franka_gazebo/meshes/collision/link3.stl; visual mesh filename=package://franka_gazebo/meshes/visual/link3.dae
- link panda_link4: mass None -> 2.38; geometry collision mesh filename=package://franka_gazebo/meshes/collision/link4.stl; visual mesh filename=package://franka_gazebo/meshes/visual/link4.dae
- link panda_link5: mass None -> 2.74; geometry collision mesh filename=package://franka_gazebo/meshes/collision/link5.stl; visual mesh filename=package://franka_gazebo/meshes/visual/link5.dae
- link panda_link6: mass None -> 1.55; geometry collision mesh filename=package://franka_gazebo/meshes/collision/link6.stl; visual mesh filename=package://franka_gazebo/meshes/visual/link6.dae
- link panda_link7: mass None -> 0.54; geometry collision mesh filename=package://franka_gazebo/meshes/collision/link7.stl; visual mesh filename=package://franka_gazebo/meshes/visual/link7.dae
- link panda_rightfinger: mass None -> 0.1; geometry collision mesh filename=package://franka_gazebo/meshes/collision/finger.stl; visual mesh filename=package://franka_gazebo/meshes/visual/finger.dae
Joints:
- added joint panda_joint_world: type fixed, parent world, child panda_link0, origin xyz=0 0 0 rpy=0 0 0
- joint panda_finger_joint1: limit lower=0.0 upper=0.04 effort=20 velocity=0.2 -> lower=-0.001 upper=0.04 effort=20 velocity=0.3
- joint panda_finger_joint2: axis 0 1 0 -> 0 -1 0; limit lower=0.0 upper=0.04 effort=20 velocity=0.2 -> lower=-0.001 upper=0.04 effort=20 velocity=0.3; mimic joint=panda_finger_joint1 -> (none)
- joint panda_joint4: limit lower=-3.0718 upper=-0.0698 effort=87 velocity=2.1750 -> lower=-3.0718 upper=0.0698 effort=87 velocity=2.1750
