Commit message: update spot arm urdf

File: configs/urdfs/spot_arm.urdf (robot description, URDF)
Before this commit: robot spot_arm, 10 links, 9 joints
Joints:
- joint arm_joint1: origin xyz=0.0 0.0 0.065 rpy=0 0 0 -> xyz=0.0 0.0 0.065 rpy=0 0 1.5707963267948966
- joint arm_joint2: axis -1.0 0.0 0.0 -> 1.0 0.0 0.0; origin xyz=0.015 0.0 0.05 rpy=0 0 0 -> xyz=0.015 0.0 0.05 rpy=-3.141592653589793 0 0
